File: hardware/step_counter_pcb/step_counter_pcb.kicad_sch (KiCad schematic)
At the start: 13 parts, among them J1 LiPo_Battery, SW1 SW_SPST, U1 TPS63031DSK, U2 ESP32-C6-MINI-1

Commit message: Cleaned up Power block
Parts:
- removed TP4: TestPoint, symbol Connector:TestPoint
- removed U2: ESP32-C6-MINI-1, RF_Module:ESP32-C6-MINI-1, symbol RF_Module:ESP32-C6-MINI-1
- added NT1: NetTie_2, symbol Device:NetTie_2
- C2: value 10 uF -> 0.1uF
- C3: value 0.1 uF -> 10 uF
- L1: value 1.5uH -> 1.5 uH
- TP2: value TestPoint -> VBAT_SW
- TP3: value TestPoint -> 3V3
Connections:
- net 3V3: now also C3.1; no longer C2.1
- net GNDPWR: now also C3.2, U1.9 (GND), NT1.2; no longer C2.2
- net GNDREF: now also C2.2, NT1.1; no longer C3.2, U1.9 (GND)
- net VBAT_SW: now also C2.1, U1.6 (EN), U1.7 (PS/SYNC), U1.8 (VINA)
- net VBAT renamed VBAT+

Commit message: Adds controller block
Parts:
- removed SW1: SW_SPST, symbol Switch:SW_SPST
- added J2: USB_C_Receptacle_USB2.0_16P, symbol Connector:USB_C_Receptacle_USB2.0_16P
- added R1: 10k, symbol Device:R_US
- added R2, R3: 33, symbol Device:R_US
- added R4, R5: R_US, symbol Device:R_US
- added SW1, SW2: SW_Push, symbol Switch:SW_Push
- added U2: ESP32-C3-MINI-1, PCM_Espressif:ESP32-C3-MINI-1, symbol PCM_Espressif:ESP32-C3-MINI-1
- added U3: LIS2DUX12, LGA-12_2.0X2.0X0.74_LIS2DUX12_STM, symbol 2026-10-17_22-18-52:LIS2DUX12
- TP3: value 3V3 -> TestPoint
Connections:
- net 3V3: now also R1.1, U2.3 (3V3)
- net GND: now also J2.A1 (GND), J2.A12 (GND), J2.B1 (GND), J2.B12 (GND), J2.SH (SHIELD), R4.2, R5.2, SW2.1, U2.1 (GND), U2.11 (GND), U2.14 (GND), U2.2 (GND), U2.36 (GND), U2.37 (GND), U2.38 (GND), U2.39 (GND), U2.40 (GND), U2.41 (GND), U2.42 (GND), U2.43 (GND), U2.44 (GND), U2.45 (GND), U2.46 (GND), U2.47 (GND), U2.48 (GND), U2.49 (GND), U2.50 (GND), U2.51 (GND), U2.52 (GND), U2.53 (GND), U3.6 (GND), U3.8 (GND)
- net VBAT+: now also SW1.1
- net VBAT_SW: now also SW1.2
- new net: J2.A6 (D+), J2.B6 (D+), R2.1
- new net: R2.2, U2.27 (GPIO19/USB_D+)
- new net: R1.2, SW2.2, U2.8 (EN/CHIP_PU)
- new net: R3.2, U2.26 (GPIO18/USB_D-)
- new net: J2.A7 (D-), J2.B7 (D-), R3.1
- new net: J2.A4 (VBUS), J2.A9 (VBUS), J2.B4 (VBUS), J2.B9 (VBUS)
- new net: J2.A5 (CC1), R5.1
- new net: J2.B5 (CC2), R4.1
- new net ACC_INT1: U2.6 (GPIO3/ADC1_CH3)
- new net I2C_SDA: U2.18 (GPIO4/ADC1_CH4)
- new net LCD_A0: U2.12 (GPIO0/ADC1_CH0/XTAL_32K_P)
- new net LCD_CS: U2.16 (GPIO10)
- new net LCD_MOSI: U2.21 (GPIO7)
- new net LCD_RESET: U2.13 (GPIO1/ADC1_CH1/XTAL_32K_N)
- new net LCD_SCK: U2.20 (GPIO6)
- no-connect marks 0 -> 9
Other:
- company: (none) -> Mathew Nacev
- title: (none) -> Main Schematic for Step Tracker
- moved on the sheet: C1, C2, C3, C4, J1, L1, NT1, TP1, TP2, U1

Commit message: This commit finishes the first revision of the schematic and updates the documentation
Parts:
- removed SW1: SW_Push, symbol Switch:SW_Push
- added C5, C7: 100 nF, symbol Device:C
- added C6: 10 uF, symbol Device:C
- added C8: C, symbol Device:C
- added C9: 0.1 uF, symbol Device:C
- added R10, R11, R6, R7: 4.7 k, symbol Device:R_US
- added R8, R9: R_US, symbol Device:R_US
- added SW1: SW_SPST, symbol Switch:SW_SPST
- added U4: EEPROM, Package_DFN_QFN:DFN-8-1EP_3x2mm_P0.5mm_EP1.3x1.5mm, symbol Memory_EEPROM:AT24CS32-MAHM
- added U5: ER_OLEDM0.91_1x-I2C, Display:ER_OLEDM0.91_1x-I2C, symbol Display_Graphic:ER_OLEDM0.91_1x-I2C
- C3, C4: value 10 uF -> 11 uF
Connections:
- net 3V3: now also U3.10 (VDD_IO), U3.2 (CS), U3.9 (VDD), C5.2, C6.1, C7.1, C8.2, R10.1, R11.2, R6.2, R7.1, R8.1, R9.2, U4.8 (VCC), U5.2 (VCC)
- net ACC_INT1: now also U3.12 (INT1)
- net GND: now also U3.3 (SDO/SA0), U3.7 (RES), C5.1, C6.2, C7.2, C8.1, C9.1, U4.1 (A0), U4.2 (A1), U4.3 (A2), U4.4 (GND), U4.7 (WP), U4.9 (GND), U5.1 (GND)
- net I2C_SDA: now also U3.4 (SDA/SDI/SDO), R11.1, R6.1, R8.2, U4.5 (SDA), U5.4 (SDA)
- net VBAT+: now also SW1.1 (A)
- net VBAT_SW: now also C9.2, SW1.2 (B); no longer C2.1, U1.6 (EN), U1.7 (PS/SYNC)
- net I2C_SCL: now reaches U2.19 (GPIO5/ADC2_CH0)
- net I2C_SCL: now also U3.1 (SCL/SPC), R10.2, R7.2, R9.1, U4.6 (SCL), U5.3 (SCL)
- net LCD_A0: no longer names the net of U2.12 (GPIO0/ADC1_CH0/XTAL_32K_P)
- net LCD_CS: no longer names the net of U2.16 (GPIO10)
- net LCD_MOSI: no longer names the net of U2.21 (GPIO7)
- net LCD_RESET: no longer names the net of U2.13 (GPIO1/ADC1_CH1/XTAL_32K_N)
- net LCD_SCK: no longer names the net of U2.20 (GPIO6)
- new net: C2.1, U1.6 (EN), U1.7 (PS/SYNC)
- no-connect marks 9 -> 14
Other:
- moved on the sheet: U3

Commit message: Finalizes schematic and assigns footprints
Parts:
- removed C2: 0.1uF, symbol Device:C
- removed NT1: NetTie_2, symbol Device:NetTie_2
- removed R10, R11: 4.7 k, symbol Device:R_US
- removed R8, R9: R_US, symbol Device:R_US
- removed SW1: SW_SPST, symbol Switch:SW_SPST
- added SW3: SW_SPDT, symbol Switch:SW_SPDT
- added U6: TPD2EUSB30, Package_TO_SOT_SMD:Texas_DRT-3, symbol Power_Protection:TPD2EUSB30
- C1, C6: footprint (none) -> Capacitor_SMD:C_0805_2012Metric
- C3, C4: value 11 uF -> 10 uF; footprint (none) -> Capacitor_SMD:C_0805_2012Metric
- C5, C7, C9: footprint (none) -> Capacitor_SMD:C_0603_1608Metric
- C8: value C -> 100 nF; footprint (none) -> Capacitor_SMD:C_0603_1608Metric
- J1: footprint (none) -> Connector_JST:JST_PH_S2B-PH-K_1x02_P2.00mm_Horizontal
- J2: footprint (none) -> Connector_USB:USB_C_Receptacle_GCT_USB4105-xx-A_16P_TopMnt_Horizontal
- L1: footprint (none) -> Inductor_SMD:L_Coilcraft_LPS3010
- R1, R2, R3, R6, R7: footprint (none) -> Resistor_SMD:R_0603_1608Metric
- R4, R5: value R_US -> 5.1 k; footprint (none) -> Resistor_SMD:R_0603_1608Metric
- SW2: footprint (none) -> Button_Switch_THT:SW_PUSH_6mm
- TP1, TP2, TP3: footprint (none) -> TestPoint:TestPoint_Pad_1.0x1.0mm
- U3: footprint LGA-12_2.0X2.0X0.74_LIS2DUX12_STM -> footprints:LGA-12_2.0X2.0X0.74_LIS2DUX12_STM
Connections:
- net GNDPWR is gone; now on net GND: C1.2, C3.2, C4.2, U1.11 (PGND), U1.3 (PGND), U1.9 (GND)
- net GND: now also U1.7 (PS/SYNC), U6.3 (GND)
- net VBAT+: now also SW3.2 (B)
- net VBAT_SW: now also U1.6 (EN), SW3.1 (A)
- net at J2.A6 (D+), J2.B6 (D+), R2.1: now also U6.1 (D+)
- net at J2.A7 (D-), J2.B7 (D-), R3.1: now also U6.2 (D-)
- no-connect marks 14 -> 15
Other:
- note added: "Accerlometer Circuit"
- note added: "Controller Circuit"
- note added: "Display Circuit"
- note added: "Memory Circuit"
- note added: "Power Regulation Circuit"

Commit message: Starts layout of PCB
Parts:
- removed SW3: SW_SPDT, symbol Switch:SW_SPDT
- added SW1: SW_SPST, Button_Switch_THT:SW_CW_GPTS203211B, symbol Switch:SW_SPST
Connections:
- net VBAT+: now also SW1.1 (A)
- net VBAT_SW: now also SW1.2 (B)
- no-connect marks 15 -> 14
Changed lines of the file:
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@@
 	)
 	(no_connect
-		(at 62.23 30.48)
-	)
-	(no_connect
 		(at 238.76 88.9)
 	)
@@
 	(wire
 		(pts
-			(xy 62.23 25.4) (xy 62.23 27.94)
-		)
-		(stroke
-			(width 0)
-			(type default)
-		)
-	)
-	(wire
-		(pts
 			(xy 110.49 38.1) (xy 101.6 38.1)
 		)
@@
 	)
 	(symbol
+		(lib_id "Switch:SW_SPST")
+		(at 57.15 27.94 0)
+		(unit 1)
+		(body_style 1)
+		(exclude_from_sim no)
+		(in_bom yes)
+		(on_board yes)
+		(in_pos_files yes)
+		(dnp no)
+		(fields_autoplaced yes)
+		(property "Reference" "SW1"
+			(at 57.15 21.59 0)
+			(show_name no)
+			(do_not_autoplace no)
+			(effects
+				(font
+					(size 1.27 1.27)
+				)
+			)
+		)
+		(property "Value" "SW_SPST"
+			(at 57.15 24.13 0)
+			(show_name no)
+			(do_not_autoplace no)
+			(effects
+				(font
+					(size 1.27 1.27)
+				)
+			)
+		)
+		(property "Footprint" "Button_Switch_THT:SW_CW_GPTS203211B"
+			(at 57.15 27.94 0)
+			(hide yes)
+			(show_name no)
+			(do_not_autoplace no)
+			(effects
+				(font
+					(size 1.27 1.27)
+				)
+			)
+		)
+		(property "Datasheet" ""
+			(at 57.15 27.94 0)
+			(hide yes)
+			(show_name no)
+			(do_not_autoplace no)
+			(effects
+				(font
+					(size 1.27 1.27)
+				)
+			)
+		)
+		(property "Description" "Single Pole Single Throw (SPST) switch"
+			(at 57.15 27.94 0)
+			(hide yes)
+			(show_name no)
+			(do_not_autoplace no)
+			(effects
+				(font
+					(size 1.27 1.27)
+				)
+			)
+		)
+		(pin "2"
+		)
+		(pin "1"
+		)
+		(instances
+			(project "step_counter_pcb"
+				(path "/d4ae97c4-0375-41e9-8abd-bc197a3cb961"
+					(reference "SW1")
+					(unit 1)
+				)
+			)
+		)
+	)
+	(symbol
 		(lib_id "Device:R_US")
 		(at 44.45 97.79 0)
@@
 					(unit 1)
 				)
-			)
-		)
-	)
-	(symbol
-		(lib_id "Switch:SW_SPDT")
-		(at 57.15 27.94 0)
-		(unit 1)
-		(body_style 1)
-		(exclude_from_sim no)
-		(in_bom yes)
-		(on_board yes)
-		(in_pos_files yes)
-		(dnp no)
-		(fields_autoplaced yes)
-		(property "Reference" "SW3"
-			(at 57.15 19.05 0)
-			(show_name no)
-			(do_not_autoplace no)
-			(effects
-				(font
-					(size 1.27 1.27)
-				)
-			)
-		)
-		(property "Value" "SW_SPDT"
-			(at 57.15 21.59 0)
-			(show_name no)
-			(do_not_autoplace no)
-			(effects
-				(font
-					(size 1.27 1.27)
-				)
-			)
-		)
-		(property "Footprint" ""
-			(at 57.15 27.94 0)
-			(hide yes)
-			(show_name no)
-			(do_not_autoplace no)
-			(effects
-				(font
-					(size 1.27 1.27)
-				)
-			)
-		)
-		(property "Datasheet" ""
-			(at 57.15 35.56 0)
-			(hide yes)
-			(show_name no)
-			(do_not_autoplace no)
-			(effects
-				(font
-					(size 1.27 1.27)
-				)
-			)
-		)
-		(property "Description" "Switch, single pole double throw"
-			(at 57.15 27.94 0)
-			(hide yes)
-			(show_name no)
-			(do_not_autoplace no)
-			(effects
-				(font
-					(size 1.27 1.27)
-				)
-			)
-		)
-		(pin "2"
-		)
-		(pin "3"
-		)
-		(pin "1"
-		)
-		(instances
-			(project "step_counter_pcb"
-				(path "/d4ae97c4-0375-41e9-8abd-bc197a3cb961"
-					(reference "SW3")
-					(unit 1)
-				)
